File: mt32_keys/mt32keys.kicad_pcb (KiCad board)
At the start: 2 copper layers, 104.1 x 27.9 mm, 31 parts, among them CN4 Conn_01x02, CN5 Conn_01x07, SW11 KLS7, SW12 KLS7, SW13 KLS7, SW14 KLS7, SW15 KLS7, SW16 KLS7, SW17 KLS7, SW18 KLS7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

Commit message: Comments on dimensions added
Other:
- board text added: "Original SW board is 148 mm x 25.5 mm"
- board text added: "Original: 25.5mm"
- board text added: "Original: 27mm"
Changed lines of the file:
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@@
   (general
     (thickness 1.6)
-    (drawings 7)
+    (drawings 14)
     (tracks 136)
     (zones 0)
@@
       (net 7 /SC_0))
   )
+  (gr_text "Original: 25.5mm" (at 226.06 87.63) (layer Cmts.User)
+    (effects (font (size 1 1) (thickness 0.15)))
+  )
+  (dimension 21.59 (width 0.15) (layer Cmts.User)
+    (gr_text "21.590 mm" (at 217.2 86.995 270) (layer Cmts.User)
+      (effects (font (size 1 1) (thickness 0.15)))
+    )
+    (feature1 (pts (xy 210.82 97.79) (xy 216.486421 97.79)))
+    (feature2 (pts (xy 210.82 76.2) (xy 216.486421 76.2)))
+    (crossbar (pts (xy 215.9 76.2) (xy 215.9 97.79)))
+    (arrow1a (pts (xy 215.9 97.79) (xy 215.313579 96.663496)))
+    (arrow1b (pts (xy 215.9 97.79) (xy 216.486421 96.663496)))
+    (arrow2a (pts (xy 215.9 76.2) (xy 215.313579 77.326504)))
+    (arrow2b (pts (xy 215.9 76.2) (xy 216.486421 77.326504)))
+  )
+  (gr_text "Original: 27mm" (at 199.39 113.03) (layer Cmts.User)
+    (effects (font (size 1 1) (thickness 0.15)))
+  )
+  (dimension 21.59 (width 0.15) (layer Cmts.User)
+    (gr_text "21.590 mm" (at 200.025 109.249999) (layer Cmts.User)
+      (effects (font (size 1 1) (thickness 0.15)))
+    )
+    (feature1 (pts (xy 210.82 104.14) (xy 210.82 108.53642)))
+    (feature2 (pts (xy 189.23 104.14) (xy 189.23 108.53642)))
+    (crossbar (pts (xy 189.23 107.949999) (xy 210.82 107.949999)))
+    (arrow1a (pts (xy 210.82 107.949999) (xy 209.693496 108.53642)))
+    (arrow1b (pts (xy 210.82 107.949999) (xy 209.693496 107.363578)))
+    (arrow2a (pts (xy 189.23 107.949999) (xy 190.356504 108.53642)))
+    (arrow2b (pts (xy 189.23 107.949999) (xy 190.356504 107.363578)))
+  )
+  (gr_text "Original SW board is 148 mm x 25.5 mm" (at 123.19 110.49) (layer Cmts.User)
+    (effects (font (size 1 1) (thickness 0.15)))
+  )
+  (dimension 27.94 (width 0.15) (layer Cmts.User)
+    (gr_text "27.940 mm" (at 100.3 90.17 270) (layer Cmts.User)
+      (effects (font (size 1 1) (thickness 0.15)))
+    )
+    (feature1 (pts (xy 106.68 104.14) (xy 101.013579 104.14)))
+    (feature2 (pts (xy 106.68 76.2) (xy 101.013579 76.2)))
+    (crossbar (pts (xy 101.6 76.2) (xy 101.6 104.14)))
+    (arrow1a (pts (xy 101.6 104.14) (xy 101.013579 103.013496)))
+    (arrow1b (pts (xy 101.6 104.14) (xy 102.186421 103.013496)))
+    (arrow2a (pts (xy 101.6 76.2) (xy 101.013579 77.326504)))
+    (arrow2b (pts (xy 101.6 76.2) (xy 102.186421 77.326504)))
+  )
+  (dimension 104.14 (width 0.15) (layer Cmts.User)
+    (gr_text "104.140 mm" (at 158.75 71.09) (layer Cmts.User)
+      (effects (font (size 1 1) (thickness 0.15)))
+    )
+    (feature1 (pts (xy 210.82 76.2) (xy 210.82 71.803579)))
+    (feature2 (pts (xy 106.68 76.2) (xy 106.68 71.803579)))
+    (crossbar (pts (xy 106.68 72.39) (xy 210.82 72.39)))
+    (arrow1a (pts (xy 210.82 72.39) (xy 209.693496 72.976421)))
+    (arrow1b (pts (xy 210.82 72.39) (xy 209.693496 71.803579)))
+    (arrow2a (pts (xy 106.68 72.39) (xy 107.806504 72.976421)))
+    (arrow2b (pts (xy 106.68 72.39) (xy 107.806504 71.803579)))
+  )
   (gr_text GND (at 198 83) (layer F.Cu)
